Commit message: 1

File: ROS2/install/annin_ar4_moveit_config/share/annin_ar4_moveit_config/srdf/ar.srdf.xacro (robot description, xacro)
@@ -1 +1,11 @@
-/home/max/github/VisionArm/ROS2/ar4_ros_driver/annin_ar4_moveit_config/srdf/ar.srdf.xacro
+<?xml version="1.0" encoding="UTF-8"?>
+<robot xmlns:xacro="http://wiki.ros.org/xacro" name="$(arg name)">
+  <xacro:arg name="include_gripper" default="true"/>
+  <xacro:arg name="tf_prefix" default="" />
+  <xacro:include filename="$(find annin_ar4_moveit_config)/srdf/ar_macro.srdf.xacro"/>
+  <xacro:ar_srdf tf_prefix="$(arg tf_prefix)"/>
+  <xacro:if value="$(arg include_gripper)">
+    <xacro:include filename="$(find annin_ar4_moveit_config)/srdf/ar_gripper_macro.srdf.xacro"/>
+    <xacro:ar_gripper_srdf tf_prefix="$(arg tf_prefix)"/>
+  </xacro:if>
+</robot>

File: ROS2/install/annin_ar4_moveit_config/share/annin_ar4_moveit_config/srdf/ar_gripper_macro.srdf.xacro (robot description, xacro)
@@ -1 +1,27 @@
-/home/max/github/VisionArm/ROS2/ar4_ros_driver/annin_ar4_moveit_config/srdf/ar_gripper_macro.srdf.xacro
+<?xml version="1.0" ?>
+<!--This does not replace URDF, and is not an extension of URDF.
+    This is a format for representing semantic information about the robot structure.
+    A URDF file must exist for this robot as well, where the joints and the links that are referenced are defined
+-->
+<robot xmlns:xacro="http://wiki.ros.org/xacro">
+  <xacro:macro name="ar_gripper_srdf" params="tf_prefix">
+    <group name="ar_gripper">
+      <link name="${tf_prefix}gripper_base_link" />
+      <link name="${tf_prefix}gripper_jaw1_link" />
+      <link name="${tf_prefix}gripper_jaw2_link" />
+      <joint name="${tf_prefix}gripper_jaw1_joint" />
+      <passive_joint name="${tf_prefix}gripper_jaw2_joint" />
+    </group>
+    <group_state name="open" group="ar_gripper">
+      <joint name="${tf_prefix}gripper_jaw1_joint" value="0.014" />
+    </group_state>
+    <group_state name="closed" group="ar_gripper">
+      <joint name="${tf_prefix}gripper_jaw1_joint" value="0.000" />
+    </group_state>
+    <disable_collisions link1="${tf_prefix}gripper_base_link" link2="${tf_prefix}gripper_jaw1_link" reason="Adjacent" />
+    <disable_collisions link1="${tf_prefix}gripper_base_link" link2="${tf_prefix}gripper_jaw2_link" reason="Adjacent" />
+    <disable_collisions link1="${tf_prefix}gripper_jaw1_link" link2="${tf_prefix}gripper_jaw2_link" reason="Default" />
+    <disable_collisions link1="${tf_prefix}link_6" link2="${tf_prefix}gripper_base_link" reason="Adjacent" />
+    <disable_collisions link1="${tf_prefix}link_5" link2="${tf_prefix}gripper_base_link" reason="Adjacent" />
+  </xacro:macro>
+</robot>

File: ROS2/install/annin_ar4_moveit_config/share/annin_ar4_moveit_config/srdf/ar_macro.srdf.xacro (robot description, xacro)
@@ -1 +1,43 @@
-/home/max/github/VisionArm/ROS2/ar4_ros_driver/annin_ar4_moveit_config/srdf/ar_macro.srdf.xacro
+<?xml version="1.0" ?>
+<!--This does not replace URDF, and is not an extension of URDF.
+    This is a format for representing semantic information about the robot structure.
+    A URDF file must exist for this robot as well, where the joints and the links that are referenced are defined
+-->
+<robot xmlns:xacro="http://wiki.ros.org/xacro">
+  <xacro:macro name="ar_srdf" params="tf_prefix">
+    <group name="ar_manipulator">
+      <joint name="${tf_prefix}joint_1" />
+      <joint name="${tf_prefix}joint_2" />
+      <joint name="${tf_prefix}joint_3" />
+      <joint name="${tf_prefix}joint_4" />
+      <joint name="${tf_prefix}joint_5" />
+      <joint name="${tf_prefix}joint_6" />
+      <joint name="${tf_prefix}ee_joint"/>
+    </group>
+    <group_state name="home" group="ar_manipulator">
+      <joint name="${tf_prefix}joint_1" value="0" />
+      <joint name="${tf_prefix}joint_2" value="0" />
+      <joint name="${tf_prefix}joint_3" value="0" />
+      <joint name="${tf_prefix}joint_4" value="0" />
+      <joint name="${tf_prefix}joint_5" value="0" />
+      <joint name="${tf_prefix}joint_6" value="0" />
+    </group_state>
+    <group_state name="upright" group="ar_manipulator">
+      <joint name="${tf_prefix}joint_1" value="0" />
+      <joint name="${tf_prefix}joint_2" value="-0.087" />
+      <joint name="${tf_prefix}joint_3" value="-1.4" />
+      <joint name="${tf_prefix}joint_4" value="0" />
+      <joint name="${tf_prefix}joint_5" value="0" />
+      <joint name="${tf_prefix}joint_6" value="0" />
+    </group_state>
+    <disable_collisions link1="${tf_prefix}base_link" link2="${tf_prefix}link_1" reason="Adjacent" />
+    <disable_collisions link1="${tf_prefix}link_1" link2="${tf_prefix}link_2" reason="Adjacent" />
+    <disable_collisions link1="${tf_prefix}link_1" link2="${tf_prefix}link_3" reason="Never" />
+    <disable_collisions link1="${tf_prefix}link_2" link2="${tf_prefix}link_3" reason="Adjacent" />
+    <disable_collisions link1="${tf_prefix}link_3" link2="${tf_prefix}link_4" reason="Adjacent" />
+    <disable_collisions link1="${tf_prefix}link_3" link2="${tf_prefix}link_5" reason="Never" />
+    <disable_collisions link1="${tf_prefix}link_3" link2="${tf_prefix}link_6" reason="Never" />
+    <disable_collisions link1="${tf_prefix}link_4" link2="${tf_prefix}link_5" reason="Adjacent" />
+    <disable_collisions link1="${tf_prefix}link_5" link2="${tf_prefix}link_6" reason="Adjacent" />
+  </xacro:macro>
+</robot>

File: ROS2/install/annin_ar4_moveit_config/share/annin_ar4_moveit_config/urdf/fake_ar.urdf.xacro (robot description, xacro)
@@ -1 +1,37 @@
-/home/max/github/VisionArm/ROS2/ar4_ros_driver/annin_ar4_moveit_config/urdf/fake_ar.urdf.xacro
+<?xml version="1.0"?>
+<robot xmlns:xacro="http://wiki.ros.org/xacro" name="$(arg ar_model)">
+  <xacro:include filename="$(find annin_ar4_description)/urdf/ar_macro.xacro"/>
+  <xacro:include filename="$(find annin_ar4_description)/urdf/ar_gripper_macro.xacro"/>
+  <xacro:include filename="$(find annin_ar4_description)/urdf/ar.ros2_control.xacro"/>
+  <xacro:include filename="$(find annin_ar4_description)/urdf/ar_gripper.ros2_control.xacro"/>
+  <xacro:arg name="tf_prefix" default="" />
+  <link name="world" />
+  <xacro:ar_robot
+    tf_prefix="$(arg tf_prefix)"
+    parent="world"
+    robot_parameters_file="$(find annin_ar4_description)/config/$(arg ar_model).yaml"
+  >
+    <origin xyz="0 0 0" rpy="0 0 0" />
+  </xacro:ar_robot>
+  <xacro:ar_gripper
+    tf_prefix="$(arg tf_prefix)"
+    parent="$(arg tf_prefix)ee_link"
+  />
+  <xacro:ar_ros2_control
+    ar_model="$(arg ar_model)"
+    plugin_name="mock_components/GenericSystem"
+    serial_port="/dev/ttyACM0"
+    calibrate="False"
+    robot_parameters_file="$(find annin_ar4_description)/config/$(arg ar_model).yaml"
+    joint_offset_parameters_file="$(find annin_ar4_driver)/config/joint_offsets/$(arg ar_model).yaml"
+    driver_parameters_file="$(find annin_ar4_driver)/config/driver.yaml"
+    tf_prefix="$(arg tf_prefix)"
+  />
+  <xacro:ar_gripper_ros2_control
+    name="ARGripperFakeSystem"
+    plugin_name="mock_components/GenericSystem"
+    serial_port="/dev/ttyUSB0"
+    driver_parameters_file="$(find annin_ar4_driver)/config/gripper_driver.yaml"
+    tf_prefix="$(arg tf_prefix)"
+  />
+</robot>
